File: corne-scott/pcb/corne-light.kicad_pcb (KiCad board)
At the start: 2 copper layers, 271.8 x 105.6 mm, 118 parts, among them J1 MJ-4PP-9, J2 OLED, J5 Breakaway_Tabs, J6 MJ-4PP-9, J7 OLED, SW1 SW_PUSH, SW10 SW_PUSH, SW11 SW_PUSH, SW12 SW_PUSH, SW13 SW_PUSH, SW14 SW_PUSH, SW15 SW_PUSH, SW16 SW_PUSH, SW17 SW_PUSH, SW18 SW_PUSH, SW19 SW_PUSH, SW2 SW_PUSH, SW20 SW_PUSH, SW21 SW_PUSH, SW22 SW_PUSH, SW23 SW_PUSH, SW24 SW_PUSH, SW25 SW_PUSH, SW26 SW_PUSH, SW27 SW_PUSH, SW28 SW_PUSH, SW29 SW_PUSH, SW3 SW_PUSH, SW30 SW_PUSH, SW31 SW_PUSH, SW32 SW_PUSH, SW33 SW_PUSH, SW34 SW_PUSH, SW35 SW_PUSH, SW36 SW_PUSH, SW37 SW_PUSH, SW38 SW_PUSH, SW39 SW_PUSH, SW4 SW_PUSH, SW40 SW_PUSH, SW41 SW_PUSH, SW42 SW_PUSH, SW5 SW_PUSH, SW6 SW_PUSH, SW7 SW_PUSH, SW8 SW_PUSH, SW9 SW_PUSH, U1 ProMicro, U2 ProMicro

Commit message: Remove outer row of switches
Parts:
- removed D1, D13, D22, D28, D34, D7: D, kbd:D3_TH
- removed SW1, SW13, SW22, SW28, SW34, SW7: SW_PUSH, kbd:CherryMX_1u
Routing:
- net col0_r: track 177.7 -> 0.00 mm, vias 1 -> 0
- net col0: track 171.3 -> 0.00 mm, vias 3 -> 0
- net Net-(D28-Pad2): track 12.0 -> 0.00 mm
- net Net-(D22-Pad2): track 12.0 -> 0.00 mm
- net Net-(D34-Pad2): track 12.0 -> 0.00 mm
- net row0: track 129.2 -> 121.3 mm
- net row2_r: track 115.4 -> 107.5 mm
- net row1_r: track 112.6 -> 104.7 mm
- net row0_r: track 113.6 -> 105.7 mm
- net row1: track 145.0 -> 137.2 mm
- net row2: track 135.8 -> 128.1 mm
- net Net-(D13-Pad2): track 6.78 -> 0.00 mm
- net Net-(D7-Pad2): track 6.78 -> 0.00 mm
- net Net-(D1-Pad2): track 6.78 -> 0.00 mm
