File: corne-scott/pcb/corne-light.kicad_pcb (KiCad board)
At the start: 2 copper layers, 271.8 x 105.6 mm, 106 parts, among them J1 MJ-4PP-9, J2 OLED, J5 Breakaway_Tabs, J6 MJ-4PP-9, J7 OLED, SW10 SW_PUSH, SW11 SW_PUSH, SW12 SW_PUSH, SW14 SW_PUSH, SW15 SW_PUSH, SW16 SW_PUSH, SW17 SW_PUSH, SW18 SW_PUSH, SW19 SW_PUSH, SW2 SW_PUSH, SW20 SW_PUSH, SW21 SW_PUSH, SW23 SW_PUSH, SW24 SW_PUSH, SW25 SW_PUSH, SW26 SW_PUSH, SW27 SW_PUSH, SW29 SW_PUSH, SW3 SW_PUSH, SW30 SW_PUSH, SW31 SW_PUSH, SW32 SW_PUSH, SW33 SW_PUSH, SW35 SW_PUSH, SW36 SW_PUSH, SW37 SW_PUSH, SW38 SW_PUSH, SW39 SW_PUSH, SW4 SW_PUSH, SW40 SW_PUSH, SW41 SW_PUSH, SW42 SW_PUSH, SW5 SW_PUSH, SW6 SW_PUSH, SW8 SW_PUSH, SW9 SW_PUSH, U1 ProMicro, U2 ProMicro

Commit message: Move through holes in
Parts:
- moved Ref** 19.1 mm to (246.5, 55.9)
Changed lines of the file:
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@@
     (mod_text_size 1 1)
     (mod_text_width 0.15)
-    (pad_size 0.8128 0.8128)
-    (pad_drill 0.8128)
+    (pad_size 4.8 4.8)
+    (pad_drill 4.8)
     (pad_to_mask_clearance 0.2)
     (aux_axis_origin 145.73 12.66)
@@
       (effects (font (size 1 1) (thickness 0.15)) (justify mirror))
     )
-    (pad "" thru_hole circle (at 0 0 180) (size 4.8 4.8) (drill 4.8) (layers *.Cu *.Mask))
+    (pad "" thru_hole circle (at -18.992 0.1465 180) (size 4.8 4.8) (drill 4.8) (layers *.Cu *.Mask))
   )
   (module kbd:M2_HOLE_v2 (layer B.Cu)
@@
       (effects (font (size 1 1) (thickness 0.15)) (justify mirror))
     )
-    (pad "" thru_hole circle (at 0 0 180) (size 4.8 4.8) (drill 4.8) (layers *.Cu *.Mask))
+    (pad "" thru_hole circle (at -18.992 0.1465 180) (size 4.8 4.8) (drill 4.8) (layers *.Cu *.Mask))
   )
   (module kbd:M2_HOLE_v2 (layer F.Cu)
@@
       (effects (font (size 1 1) (thickness 0.15)))
     )
-    (pad "" thru_hole circle (at 0 0) (size 4.8 4.8) (drill 4.8) (layers *.Cu *.Mask))
+    (pad "" thru_hole circle (at -19.008 -0.006) (size 4.8 4.8) (drill 4.8) (layers *.Cu *.Mask))
   )
   (module kbd:M2_HOLE_v2 (layer F.Cu)
-    (at 265.5325 55.28)
+    (at 246.4845 55.924)
     (descr "Mounting Hole 2.2mm, no annular, M2")
     (tags "mounting hole 2.2mm no annular m2")
@@
       (effects (font (size 1 1) (thickness 0.15)))
     )
-    (pad "" thru_hole circle (at 0 0) (size 4.8 4.8) (drill 4.8) (layers *.Cu *.Mask))
+    (pad "" thru_hole circle (at 0.04 -0.65) (size 4.8 4.8) (drill 4.8) (layers *.Cu *.Mask))
   )
   (module kbd:D3_TH (layer F.Cu)
