File: corne-scott/pcb/corne-light.kicad_pcb (KiCad board)
At the start: 2 copper layers, 271.8 x 105.6 mm, 118 parts, among them J1 MJ-4PP-9, J2 OLED, J5 Breakaway_Tabs, J6 MJ-4PP-9, J7 OLED, SW1 SW_PUSH, SW10 SW_PUSH, SW11 SW_PUSH, SW12 SW_PUSH, SW13 SW_PUSH, SW14 SW_PUSH, SW15 SW_PUSH, SW16 SW_PUSH, SW17 SW_PUSH, SW18 SW_PUSH, SW19 SW_PUSH, SW2 SW_PUSH, SW20 SW_PUSH, SW21 SW_PUSH, SW22 SW_PUSH, SW23 SW_PUSH, SW24 SW_PUSH, SW25 SW_PUSH, SW26 SW_PUSH, SW27 SW_PUSH, SW28 SW_PUSH, SW29 SW_PUSH, SW3 SW_PUSH, SW30 SW_PUSH, SW31 SW_PUSH, SW32 SW_PUSH, SW33 SW_PUSH, SW34 SW_PUSH, SW35 SW_PUSH, SW36 SW_PUSH, SW37 SW_PUSH, SW38 SW_PUSH, SW39 SW_PUSH, SW4 SW_PUSH, SW40 SW_PUSH, SW41 SW_PUSH, SW42 SW_PUSH, SW5 SW_PUSH, SW6 SW_PUSH, SW7 SW_PUSH, SW8 SW_PUSH, SW9 SW_PUSH, U1 ProMicro, U2 ProMicro

Commit message: Make switches hotswap
Parts:
- RSW1, RSW2: footprint kbd:ResetSW_1side -> MX_Only:MXOnly-1U-Hotswap
- SW1, SW10, SW11, SW12, SW13, SW14, SW15, SW16, SW17, SW18, SW19, SW2, SW20, SW21, SW22, SW23, SW24, SW25, SW26, SW27, SW28, SW29, SW3, SW30, SW31, SW32, SW33, SW34, SW35, SW36, SW37, SW38, SW39, SW4, SW40, SW41, SW42, SW5, SW6, SW7, SW8, SW9: footprint kbd:CherryMX_1u -> MX_Only:MXOnly-1U-Hotswap
Routing:
- net (no net): track 0.00 -> 20.6 mm
- net Net-(D42-Pad2): track 31.8 -> 31.0 mm
- net Net-(D33-Pad2): track 6.29 -> 5.69 mm
- net Net-(D31-Pad2): track 7.82 -> 7.22 mm
- net Net-(D29-Pad2): track 6.93 -> 6.32 mm
- net Net-(D27-Pad2): track 6.29 -> 5.69 mm
- net Net-(D25-Pad2): track 7.82 -> 7.22 mm
- net Net-(D23-Pad2): track 6.93 -> 6.32 mm
- net Net-(D32-Pad2): track 11.9 -> 11.3 mm
- net Net-(D30-Pad2): track 11.9 -> 11.3 mm
- net Net-(D28-Pad2): track 12.0 -> 11.4 mm
- net Net-(D26-Pad2): track 11.9 -> 11.3 mm
- net Net-(D24-Pad2): track 11.9 -> 11.3 mm
- net Net-(D22-Pad2): track 12.0 -> 11.4 mm
- net Net-(D34-Pad2): track 12.0 -> 11.4 mm
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